File: PCB/motorControlBoard.kicad_sch (KiCad schematic)
At the start: 12 parts, among them J1 Barrel_Jack, J2 B5B-XH-ALFSN, J3 B5B-XH-ALFSN, J4 B5B-XH-ALFSN, U1 ULN2003A, U2 ULN2003A, U3 ULN2003A

Commit message: final (i think)
Parts:
- removed C3: 100nF, Capacitor_THT:C_Disc_D5.0mm_W2.5mm_P5.00mm, symbol Device:C_Small
- removed U3: ULN2003A, Package_DIP:DIP-16_W7.62mm, symbol Transistor_Array:ULN2003A
- added D1: LED, LED_THT:LED_D5.0mm, symbol Device:LED
- added R1: 220 Ohm, Resistor_THT:R_Axial_DIN0204_L3.6mm_D1.6mm_P7.62mm_Horizontal, symbol Device:R_US
Connections:
- net GND: now also R1.2
- net at A1.30 (VIN), C1.1, C2.1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: now also D1.2 (A)
- net at U2.12 (O5): now also J4.4
- net at U2.5 (I5): now also A1.19 (A0)
- net at J4.1: now also U1.12 (O5)
- net at J4.2: now also U1.11 (O6)
- net at J4.3: now also U1.10 (O7)
- net at U1.5 (I5): now also A1.20 (A1)
- net at U1.6 (I6): now also A1.21 (A2)
- net at U1.7 (I7): now also A1.22 (A3)
- new net: D1.1 (K), R1.1
Other:
- moved on the sheet: J1, U1, U2
